File: KiCad/PPP.sch (KiCad schematic (older format))
At the start: 117 parts, among them P1 5V, P10 CONN_8X2, P11 CONN_8X2, P12 CONN_8X2, P13 CONN_8X2, P14 CONN_8X2, P15 CONN_8X2, P16 CONN_8X2, P17 CONN_8X2, P18 CONN_8X2, P19 CONN_4X2, P2 INT/~INT, P20 CONN_8X2, P21 CONN_8X2, P22 CONN_8X2, P23 CONN_8X2, P24 CONN_8X2, P25 CONN_8X2, P26 CONN_8X2, P27 CONN_8X2, P28 CONN_8X2, P29 CONN_4X2, P3 PROP_PLUG, P30 CONN_8X2, P31 CONN_8X2, P32 CONN_8X2, P33 CONN_8X2, P34 CONN_8X2, P35 CONN_8X2, P36 CONN_8X2, P37 CONN_8X2, P38 CONN_8X2, P39 CONN_4X2, P4 PORT_B, P40 CONN_8X2, P41 CONN_8X2, P42 CONN_8X2, P43 CONN_8X2, P44 CONN_8X2, P45 CONN_8X2, P46 CONN_8X2, P47 CONN_8X2, P48 CONN_8X2, P49 CONN_4X2, P5 PARALLEL, P50 CONN_4X2, P51 CONN_8X2, P52 CONN_8X2, P53 CONN_8X2, P54 CONN_8X2, P55 CONN_8X2, P56 CONN_8X2, P57 CONN_8X2, P58 CONN_8X2, P59 CONN_2X2, P6 KEYBOARD, P60 CONN_2X2, P61 CONN_8X2, P62 CONN_8X2, P63 CONN_8X2, P64 CONN_4X2, P7 SERIAL, P8 VGA, P9 SD_CARD, U1 74LS06, U2 MAX232, U3 LM3940, U4 P8X32A, U5 24C512, X1 5MHz

Commit message: Add 1.1 files
Signed-off-by: Sergey Kiselev <skiselev@gmail.com>
Parts:
- removed P10, P11, P12, P13, P14, P15, P16, P17, P18, P20, P21, P22, P23, P24, P25, P26, P27, P28, P30, P31, P32, P33, P34, P35, P36, P37, P38, P40, P41, P42, P43, P44, P45, P46, P47, P48, P51, P52, P53, P54, P55, P56, P57, P58, P61, P62, P63: CONN_8X2, symbol CONN_8X2
- removed P19, P29, P39, P49, P50, P64: CONN_4X2, symbol CONN_4X2
- removed P59, P60: CONN_2X2, symbol CONN_2X2
- added C14: 100uF, symbol CP1
- added P10, P11, P12, P13, P14, P15, P16, P17, P18, P20, P21, P22, P23, P24, P25, P26, P27, P28, P30, P31, P32, P33, P34, P35, P36, P37, P38, P40, P41, P42, P43, P44, P45, P46, P47, P48, P51, P52, P53, P54, P55, P56, P57, P58, P61, P62, P63: PROTO_4X4, symbol PROTO_4X4
- added P19, P29, P39, P49, P50, P64: PROTO_2X4, symbol PROTO_2X4
- added P59, P60: PROTO_2X2, symbol PROTO_2X2
- C13: renamed from C12; value 10uF -> 100uF
- renumbered C13 to C12
Connections:
- net GND: now also C14.2, P17.13, P17.14, P17.15, P17.16, P27.13, P27.14, P27.15, P27.16, P38.13, P38.14, P38.15, P38.16, P48.13, P48.14, P48.15, P48.16, P59.3, P59.4, P64.5, P64.6, P64.7, P64.8
- net VCC: now also P10.1, P10.2, P10.3, P10.4, P20.1, P20.2, P20.3, P20.4, P30.1, P30.2, P30.3, P30.4, P39.4, P39.8, P40.1, P40.2, P40.3, P40.4, P53.1, P53.2, P53.3, P53.4, P60.1, P60.2
- net VDD: now also C14.1
- no-connect marks 779 -> 776
Other:
- moved on the sheet: C1, C11, C13, C2, C3, C4, C5, HOLE1, HOLE2, HOLE3, HOLE4, P1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
